Commit message: Added Novatel Smart6 GPS accessory and updated localization to use IMU.

File: warthog_description/urdf/accessories.urdf.xacro (robot description, xacro)
@@ -9,3 +9,14 @@
     warthog_base/launch/base.launch
   -->
+  <!-- If enabled, generate a Novatel Smart6 payload. -->
+  <xacro:include filename="accessories/novatel_smart6.urdf.xacro" />
+  <xacro:if value="$(optenv WARTHOG_NAVSAT_SMART6 0)">
+    <novatel_smart6 prefix="$(optenv WARTHOG_NAVSAT_SMART6_MOUNT navsat)"/>
+    <joint name="$(optenv WARTHOG_NAVSAT_SMART6_MOUNT navsat)_joint" type="fixed">
+    <origin xyz="$(optenv WARTHOG_NAVSAT_SMART6_OFFSET 0 0 0)"
+            rpy="$(optenv WARTHOG_NAVSAT_SMART6_RPY 0 0 0)" />
+      <parent link="top_chassis_link" />
+      <child link="$(optenv WARTHOG_NAVSAT_SMART6_MOUNT navsat)_link" />
+    </joint>
+  </xacro:if>
 </robot>

File: warthog_description/urdf/warthog.urdf.xacro (robot description, xacro)
@@ -126,8 +126,10 @@
     </collision>
   </link>
-  <gazebo reference="chassis_link">
-    <selfCollide>false</selfCollide>
-    <material>Gazebo/Black</material>
-  </gazebo>
+  <link name="top_chassis_link"></link>
+  <joint name="top_link_joint" type="fixed">
+    <origin xyz="0 0 ${chassis_height/2}" rpy="0 0 0" />
+    <parent link="chassis_link"/>
+    <child link="top_chassis_link" />
+  </joint>
   <!-- This link is purely to complete the visual look -->
   <link name="diff_link">
@@ -154,12 +156,9 @@
     </visual>
   </link>
-  <joint name="$diff_link_jnt" type="fixed">
+  <joint name="diff_link_jnt" type="fixed">
     <parent link="chassis_link"/>
     <child link="diff_link"/>
     <origin xyz="-0.65 0 0.07" rpy="0 0 0" />
   </joint>
-  <gazebo reference="diff_link">
-    <material>Gazebo/Grey</material>
-  </gazebo>
   <!-- Bring in simulation data for Gazebo. -->
   <xacro:include filename="$(find warthog_description)/urdf/warthog.gazebo" />

Commit message: Completely redid most meshes and added the bulkhead and arm mounting point. Added configs for both as well. Took meshes from 4 Mb down to 1 (total)

File: warthog_description/urdf/accessories.urdf.xacro (robot description, xacro)
@@ -20,3 +20,26 @@
     </joint>
   </xacro:if>
+  <xacro:include filename="accessories/warthog_bulkhead.urdf.xacro" />
+  <xacro:if value="$(optenv WARTHOG_BULKHEAD 0)">
+    <warthog_bulkhead/>
+    <joint name="bulkhead_link_joint" type="fixed">
+      <origin xyz="0.00705 0 0.24184" rpy="0 0 0" />
+      <parent link="top_chassis_link"/>
+      <child link="bulkhead_link" />
+    </joint>
+    <joint name="bulkhead_front_mount_link_joint" type="fixed">
+      <origin xyz="0.33987 0 0.0" rpy="0 0 0" />
+      <parent link="bulkhead_link"/>
+      <child link="bulkhead_front_mount_link" />
+    </joint>
+        <xacro:include filename="accessories/warthog_arm_mount.urdf.xacro" />
+        <xacro:if value="$(optenv WARTHOG_ARM_MOUNT 0)">
+          <warthog_arm_mount/>
+          <joint name="arm_mount_link_joint" type="fixed">
+            <origin xyz="0 0 0.02" rpy="0 0 0" />
+            <parent link="bulkhead_front_mount_link"/>
+            <child link="arm_mount_link" />
+          </joint>
+        </xacro:if>
+  </xacro:if>
 </robot>

File: warthog_description/urdf/warthog.urdf.xacro (robot description, xacro)
@@ -4,6 +4,8 @@
   <material name="dark_grey"><color rgba="0.2 0.2 0.2 1.0" /></material>
   <material name="light_grey"><color rgba="0.4 0.4 0.4 1.0" /></material>
-  <material name="yellow"><color rgba="0.8 0.8 0.0 1.0" /></material>
+  <material name="yellow"><color rgba="0.95 0.816 0.082 1.0" /></material>
   <material name="black"><color rgba="0.15 0.15 0.15 1.0" /></material>
+  <material name="white"><color rgba="0.9 0.9 0.9 1.0" /></material>
+  <material name="red"><color rgba="0.9 0.0 0.0 1.0" /></material>
   <xacro:macro name="wheel" params="prefix side fwd left">
     <link name="${prefix}_wheel">
@@ -14,5 +16,5 @@
       </inertial>
       <visual>
-        <origin xyz="0 0 0" rpy="0 0 ${PI/2}"/>
+        <origin xyz="0 0 0" rpy="0 0 ${side*PI/2}"/>
         <geometry>
           <mesh filename="package://warthog_description/meshes/wheel.stl" />
@@ -21,5 +23,5 @@
       </visual>
       <collision>
-        <origin xyz="0 0 0" rpy="${PI/2} 0 0"/>
+        <origin xyz="0 0 0" rpy="${side*PI/2} 0 0"/>
         <geometry>
           <cylinder radius="${wheel_radius}" length="${wheel_width}"/>
@@ -71,14 +73,35 @@
       </inertial>
       <visual>
-        <origin xyz="0 ${side*-1*0.05} 0.197" rpy="${PI/2} 0 ${PI/2-side*PI/2}"/>
+        <origin xyz="0 0 0" rpy="0 0 ${side*PI/2}"/>
         <geometry>
           <mesh filename="package://warthog_description/meshes/rocker.stl" />
         </geometry>
-        <material name="yellow" />
+        <material name="black"><color rgba="0.15 0.15 0.15 1.0" /></material>
+      </visual>
+      <visual>
+        <origin xyz="0 0 0" rpy="0 0 ${side*PI/2}"/>
+        <geometry>
+          <mesh filename="package://warthog_description/meshes/fenders.stl" />
+        </geometry>
+        <material name="yellow"><color rgba="0.95 0.816 0.082 1.0" /></material>
+      </visual>
+      <visual>
+        <origin xyz="0 ${side*-0.0244} 0" rpy="0 0 0"/>
+        <geometry>
+          <mesh filename="package://warthog_description/meshes/light.stl" />
+        </geometry>
+        <material name="white"><color rgba="0.9 0.9 0.9 1.0" /></material>
+      </visual>
+      <visual>
+        <origin xyz="0 ${side*-0.0244} 0" rpy="0 0 ${side*PI}"/>
+        <geometry>
+          <mesh filename="package://warthog_description/meshes/light.stl" />
+        </geometry>
+        <material name="red"><color rgba="0.9 0.0 0.0 1.0" /></material>
       </visual>
       <collision>
-        <origin xyz="0 0 0.197" rpy="0 0 0"/>
-        <geometry>
-          <box size="${diff_unit_length} ${diff_unit_width} ${diff_unit_height}"/>
+        <origin xyz="0 0 0" rpy="0 0 ${side*PI/2}"/>
+        <geometry>
+          <mesh filename="package://warthog_description/meshes/fenders.stl" />
         </geometry>
       </collision>
@@ -101,5 +124,5 @@
   <link name="base_link"></link>
   <joint name="base_link_joint" type="fixed">
-    <origin xyz="0 0 0" rpy="0 0 0" />
+    <origin xyz="0 0 0.025" rpy="0 0 0" />
     <parent link="base_link"/>
     <child link="chassis_link" />
@@ -117,10 +140,17 @@
         <mesh filename="package://warthog_description/meshes/chassis.stl" />
       </geometry>
-      <material name="black" />
+      <material name="black"><color rgba="0.15 0.15 0.15 1.0" /></material>
+    </visual>
+    <visual>
+      <origin xyz="0 0 0" rpy="0 0 0"/>
+      <geometry>
+        <mesh filename="package://warthog_description/meshes/e-stop.stl" />
+      </geometry>
+      <material name="red"><color rgba="0.9 0.0 0.0 1.0" /></material>
     </visual>
     <collision>
       <origin xyz="0 0 0" rpy="0 0 0"/>
       <geometry>
-        <box size="${chassis_length} ${chassis_width} ${chassis_height}"/>
+        <mesh filename="package://warthog_description/meshes/chassis-collision.stl" />
       </geometry>
     </collision>
@@ -128,5 +158,5 @@
   <link name="top_chassis_link"></link>
   <joint name="top_link_joint" type="fixed">
-    <origin xyz="0 0 ${chassis_height/2}" rpy="0 0 0" />
+    <origin xyz="0 0 0.27218" rpy="0 0 0" />
     <parent link="chassis_link"/>
     <child link="top_chassis_link" />
@@ -135,5 +165,5 @@
   <link name="diff_link">
     <visual>
-      <origin xyz="0 0 0" rpy="0 0 ${PI/2}"/>
+      <origin xyz="0 0 0" rpy="0 0 0"/>
       <geometry>
         <mesh filename="package://warthog_description/meshes/diff-link.stl" />
@@ -142,5 +172,5 @@
     </visual>
     <visual>
-      <origin xyz="0.285 0.3845 0.008" rpy="0 ${PI/2} 0"/>
+      <origin xyz="0 0 0" rpy="0 0 0"/>
       <geometry>
         <mesh filename="package://warthog_description/meshes/susp-link.stl" />
@@ -149,5 +179,5 @@
     </visual>
     <visual>
-      <origin xyz="0.285 -0.3845 0.008" rpy="0 ${PI/2} 0"/>
+      <origin xyz="0 0 0" rpy="0 0 0"/>
       <geometry>
         <mesh filename="package://warthog_description/meshes/susp-link.stl" />
@@ -159,5 +189,5 @@
     <parent link="chassis_link"/>
     <child link="diff_link"/>
-    <origin xyz="-0.65 0 0.07" rpy="0 0 0" />
+    <origin xyz="-0.5826 0 0.24979" rpy="0 0 0" />
   </joint>
   <!-- Bring in simulation data for Gazebo. -->
