Commit message: Fixed missing right suspension link.

File: warthog_description/urdf/warthog.urdf.xacro (robot description, xacro)
@@ -141,5 +141,5 @@
     </visual>
     <visual>
-      <origin xyz="0.285 0.3845 0.008" rpy="0 ${PI/2} 0"/>
+      <origin xyz="0.285 -0.3845 0.008" rpy="0 ${PI/2} 0"/>
       <geometry>
         <mesh filename="package://warthog_description/meshes/susp-link.stl" />

Commit message: [warthog_description] Updated URDF colours and links.

File: warthog_description/urdf/warthog.urdf.xacro (robot description, xacro)
@@ -86,5 +86,5 @@
     <joint name="${prefix}_diff_unit_jnt" type="revolute">
       <limit upper="0.15" lower="-0.15" effort="100000" velocity="1"/>
-      <parent link="base_link"/>
+      <parent link="chassis_link"/>
       <child link="${prefix}_diff_unit_link"/>
       <origin xyz="${diff_unit_offset_x} ${diff_unit_offset_y*side} ${diff_unit_offset_z}" rpy="0 0 0" />
@@ -94,10 +94,16 @@
     <gazebo reference="${prefix}_diff_unit_link">
       <selfCollide>false</selfCollide>
-      <material>Gazebo/Orange</material>
+      <material>Gazebo/Yellow</material>
     </gazebo>
   </xacro:macro>
   <xacro:diff_unit prefix="left" side="1" left="true"/>
   <xacro:diff_unit prefix="right" side="-1" left="false"/>
-  <link name="base_link">
+  <link name="base_link"></link>
+  <joint name="base_link_joint" type="fixed">
+    <origin xyz="0 0 0" rpy="0 0 0" />
+    <parent link="base_link"/>
+    <child link="chassis_link" />
+  </joint>
+  <link name="chassis_link">
     <inertial>
       <origin xyz="0 0 0" rpy="0 0 0"/>
@@ -120,7 +126,7 @@
     </collision>
   </link>
-  <gazebo reference="base_link">
+  <gazebo reference="chassis_link">
     <selfCollide>false</selfCollide>
-    <material>Gazebo/Orange</material>
+    <material>Gazebo/Black</material>
   </gazebo>
   <!-- This link is purely to complete the visual look -->
@@ -149,5 +155,5 @@
   </link>
   <joint name="$diff_link_jnt" type="fixed">
-    <parent link="base_link"/>
+    <parent link="chassis_link"/>
     <child link="diff_link"/>
     <origin xyz="-0.65 0 0.07" rpy="0 0 0" />

Commit message: Changed the URDF_EXTRAS variable so it is more flexible for external packages

File: warthog_description/urdf/warthog.urdf.xacro (robot description, xacro)
@@ -4,5 +4,5 @@
   <material name="dark_grey"><color rgba="0.2 0.2 0.2 1.0" /></material>
   <material name="light_grey"><color rgba="0.4 0.4 0.4 1.0" /></material>
-  <material name="yellow"><color rgba="0.95 0.816 0.082 1.0" /></material>
+  <material name="yellow"><color rgba="0.8 0.8 0.0 1.0" /></material>
   <material name="black"><color rgba="0.15 0.15 0.15 1.0" /></material>
   <material name="white"><color rgba="0.9 0.9 0.9 1.0" /></material>
@@ -84,5 +84,5 @@
           <mesh filename="package://warthog_description/meshes/fenders.stl" />
         </geometry>
-        <material name="yellow"><color rgba="0.95 0.816 0.082 1.0" /></material>
+        <material name="yellow"><color rgba="0.8 0.8 0.0 1.0" /></material>
       </visual>
       <visual>
@@ -124,5 +124,5 @@
   <link name="base_link"></link>
   <joint name="base_link_joint" type="fixed">
-    <origin xyz="0 0 0.025" rpy="0 0 0" />
+    <origin xyz="0 0 0" rpy="0 0 0" />
     <parent link="base_link"/>
     <child link="chassis_link" />
@@ -158,5 +158,5 @@
   <link name="top_chassis_link"></link>
   <joint name="top_link_joint" type="fixed">
-    <origin xyz="0 0 0.27218" rpy="0 0 0" />
+    <origin xyz="0 0 ${chassis_height/2}" rpy="0 0 0" />
     <parent link="chassis_link"/>
     <child link="top_chassis_link" />
@@ -187,7 +187,7 @@
   </link>
   <joint name="diff_link_jnt" type="fixed">
-    <parent link="chassis_link"/>
+    <parent link="base_link"/>
     <child link="diff_link"/>
-    <origin xyz="-0.5826 0 0.24979" rpy="0 0 0" />
+    <origin xyz="-0.58245 0 0.27475" rpy="0 0 0" />
   </joint>
   <!-- Bring in simulation data for Gazebo. -->
@@ -198,4 +198,4 @@
   <xacro:include filename="$(find warthog_description)/urdf/accessories.urdf.xacro" />
   <!-- Optional custom includes. -->
-  <xacro:include filename="$(find warthog_description)/urdf/$(optenv WARTHOG_URDF_EXTRAS empty.urdf)" />
+  <xacro:include filename="$(optenv WARTHOG_URDF_EXTRAS empty.urdf)" />
 </robot>

Commit message: Lowered the effort and increase the limits to make the diff units more accurate

File: warthog_description/urdf/warthog.urdf.xacro (robot description, xacro)
@@ -204,5 +204,5 @@
     </link>
     <joint name="${prefix}_diff_unit_joint" type="revolute">
-      <limit upper="0.15" lower="-0.15" effort="100000" velocity="1"/>
+      <limit upper="0.4" lower="-0.4" effort="100" velocity="1"/>
       <parent link="chassis_link"/>
       <child link="${prefix}_diff_unit_link"/>

Commit message: Add the WARTHOG_COLOR envar, with options 'yellow' (default) and 'olive_green'

File: warthog_description/urdf/warthog.urdf.xacro (robot description, xacro)
@@ -21,4 +21,5 @@
   <xacro:property name="chassis_mass" value="100" />
   <xacro:property name="dummy_inertia" value="1e-09"/>
+  <xacro:property name="warthog_color" value="$(optenv WARTHOG_COLOR yellow)" />
   <xacro:macro name="wheel_inertia" params="m r h">
     <inertia ixx="${m*(3*r*r+h*h)/12}" ixy="0" ixz="0"
@@ -34,4 +35,5 @@
   <material name="light_grey"><color rgba="0.4 0.4 0.4 1.0" /></material>
   <material name="yellow"><color rgba="0.95 0.816 0.082 1.0" /></material>
+  <material name="olive_green"><color rgba="0.333 0.419 0.184 1.0" /></material>
   <material name="black"><color rgba="0.15 0.15 0.15 1.0" /></material>
   <material name="white"><color rgba="0.9 0.9 0.9 1.0" /></material>
@@ -180,5 +182,10 @@
           <mesh filename="package://warthog_description/meshes/fenders.stl" />
         </geometry>
-        <material name="yellow"><color rgba="0.95 0.816 0.082 1.0" /></material>
+        <xacro:if value="${warthog_color == 'yellow'}">
+          <material name="yellow"><color rgba="0.95 0.816 0.082 1.0" /></material>
+        </xacro:if>
+        <xacro:if value="${warthog_color == 'olive_green'}">
+          <material name="olive_green"><color rgba="0.333 0.419 0.184 1.0" /></material>
+        </xacro:if>
       </visual>
       <visual>

Commit message: Simplify the paint options, add orange and sand as additional choices based on feedback from sales on the available colours.

File: warthog_description/urdf/warthog.urdf.xacro (robot description, xacro)
@@ -21,5 +21,25 @@
   <xacro:property name="chassis_mass" value="100" />
   <xacro:property name="dummy_inertia" value="1e-09"/>
+  <!--
+    Optional paint colors.
+    Available colors:
+      - yellow (default)
+      - orange
+      - olive
+      - sand
+  -->
   <xacro:property name="warthog_color" value="$(optenv WARTHOG_COLOR yellow)" />
+  <xacro:if value="${warthog_color == 'yellow'}">
+    <xacro:property name="warthog_color_rgba" value="0.95 0.816 0.082 1.0" />
+  </xacro:if>
+  <xacro:if value="${warthog_color == 'orange'}">
+    <xacro:property name="warthog_color_rgba" value="1.0 0.48 0.0 1.0" />
+  </xacro:if>
+  <xacro:if value="${warthog_color == 'olive'}">
+    <xacro:property name="warthog_color_rgba" value="0.333 0.419 0.184 1.0" />
+  </xacro:if>
+  <xacro:if value="${warthog_color == 'sand'}">
+    <xacro:property name="warthog_color_rgba" value="0.86 0.75 0.54 1.0" />
+  </xacro:if>
   <xacro:macro name="wheel_inertia" params="m r h">
     <inertia ixx="${m*(3*r*r+h*h)/12}" ixy="0" ixz="0"
@@ -35,5 +55,4 @@
   <material name="light_grey"><color rgba="0.4 0.4 0.4 1.0" /></material>
   <material name="yellow"><color rgba="0.95 0.816 0.082 1.0" /></material>
-  <material name="olive_green"><color rgba="0.333 0.419 0.184 1.0" /></material>
   <material name="black"><color rgba="0.15 0.15 0.15 1.0" /></material>
   <material name="white"><color rgba="0.9 0.9 0.9 1.0" /></material>
@@ -182,10 +201,7 @@
           <mesh filename="package://warthog_description/meshes/fenders.stl" />
         </geometry>
-        <xacro:if value="${warthog_color == 'yellow'}">
-          <material name="yellow"><color rgba="0.95 0.816 0.082 1.0" /></material>
-        </xacro:if>
-        <xacro:if value="${warthog_color == 'olive_green'}">
-          <material name="olive_green"><color rgba="0.333 0.419 0.184 1.0" /></material>
-        </xacro:if>
+        <material name="${warthog_color}">
+          <color rgba="${warthog_color_rgba}" />
+        </material>
       </visual>
       <visual>

Commit message: Add an envar to set the paint colour of the URDF (#16)
* Add the WARTHOG_COLOR envar, with options 'yellow' (default) and 'olive_green'

* Simplify the paint options, add orange and sand as additional choices based on feedback from sales on the available colours.

File: warthog_description/urdf/warthog.urdf.xacro (robot description, xacro)
@@ -21,4 +21,25 @@
   <xacro:property name="chassis_mass" value="100" />
   <xacro:property name="dummy_inertia" value="1e-09"/>
+  <!--
+    Optional paint colors.
+    Available colors:
+      - yellow (default)
+      - orange
+      - olive
+      - sand
+  -->
+  <xacro:property name="warthog_color" value="$(optenv WARTHOG_COLOR yellow)" />
+  <xacro:if value="${warthog_color == 'yellow'}">
+    <xacro:property name="warthog_color_rgba" value="0.95 0.816 0.082 1.0" />
+  </xacro:if>
+  <xacro:if value="${warthog_color == 'orange'}">
+    <xacro:property name="warthog_color_rgba" value="1.0 0.48 0.0 1.0" />
+  </xacro:if>
+  <xacro:if value="${warthog_color == 'olive'}">
+    <xacro:property name="warthog_color_rgba" value="0.333 0.419 0.184 1.0" />
+  </xacro:if>
+  <xacro:if value="${warthog_color == 'sand'}">
+    <xacro:property name="warthog_color_rgba" value="0.86 0.75 0.54 1.0" />
+  </xacro:if>
   <xacro:macro name="wheel_inertia" params="m r h">
     <inertia ixx="${m*(3*r*r+h*h)/12}" ixy="0" ixz="0"
@@ -180,5 +201,7 @@
           <mesh filename="package://warthog_description/meshes/fenders.stl" />
         </geometry>
-        <material name="yellow"><color rgba="0.95 0.816 0.082 1.0" /></material>
+        <material name="${warthog_color}">
+          <color rgba="${warthog_color_rgba}" />
+        </material>
       </visual>
       <visual>

Commit message: Move the headlights & taillights into their own links so we can apply the correct Gazebo materials to them (otherwise the robot looks symmetrical, which is confusing). Start applying different materials to the wheel diff links, depending on the paint colour. Sand & Olive are not yet supported

File: warthog_description/urdf/warthog.urdf.xacro (robot description, xacro)
@@ -205,18 +205,4 @@
         </material>
       </visual>
-      <visual>
-        <origin xyz="0 ${side*-0.0244} 0" rpy="0 0 0"/>
-        <geometry>
-          <mesh filename="package://warthog_description/meshes/light.stl" />
-        </geometry>
-        <material name="white"><color rgba="0.9 0.9 0.9 1.0" /></material>
-      </visual>
-      <visual>
-        <origin xyz="0 ${side*-0.0244} 0" rpy="0 0 ${side*PI}"/>
-        <geometry>
-          <mesh filename="package://warthog_description/meshes/light.stl" />
-        </geometry>
-        <material name="red"><color rgba="0.9 0.0 0.0 1.0" /></material>
-      </visual>
       <collision>
         <origin xyz="0 0 0" rpy="0 0 ${side*PI/2}"/>
@@ -234,8 +220,64 @@
       <dynamics damping="100" friction="0.5"/>
     </joint>
-    <gazebo reference="${prefix}_diff_unit_link">
-      <selfCollide>false</selfCollide>
-      <material>Gazebo/Yellow</material>
+    <link name="${prefix}_diff_unit_headlight_link">
+      <visual>
+        <origin xyz="0 ${side*-0.0244} 0" rpy="0 0 0"/>
+        <geometry>
+          <mesh filename="package://warthog_description/meshes/light.stl" />
+        </geometry>
+        <material name="white"><color rgba="0.9 0.9 0.9 1.0" /></material>
+      </visual>
+    </link>
+    <joint name="${prefix}_diff_unit_headlight_joint" type="fixed">
+      <parent link="${prefix}_diff_unit_link" />
+      <child link="${prefix}_diff_unit_headlight_link" />
+      <origin xyz="0 0 0" rpy="0 0 0"/>
+    </joint>
+    <gazebo reference="${prefix}_diff_unit_headlight_link">
+      <material>Gazebo/White</material>
     </gazebo>
+    <link name="${prefix}_diff_unit_taillight_link">
+      <visual>
+        <origin xyz="0 ${side*-0.0244} 0" rpy="0 0 ${side*PI}"/>
+        <geometry>
+          <mesh filename="package://warthog_description/meshes/light.stl" />
+        </geometry>
+        <material name="red"><color rgba="0.9 0.0 0.0 1.0" /></material>
+      </visual>
+    </link>
+    <joint name="${prefix}_diff_unit_taillight_joint" type="fixed">
+      <parent link="${prefix}_diff_unit_link" />
+      <child link="${prefix}_diff_unit_taillight_link" />
+      <origin xyz="0 0 0" rpy="0 0 0"/>
+    </joint>
+    <gazebo reference="${prefix}_diff_unit_taillight_link">
+      <material>Gazebo/Red</material>
+    </gazebo>
+    <xacro:if value="${warthog_color == 'yellow'}">
+      <gazebo reference="${prefix}_diff_unit_link">
+        <selfCollide>false</selfCollide>
+        <material>Gazebo/Yellow</material>
+      </gazebo>
+    </xacro:if>
+    <xacro:if value="${warthog_color == 'orange'}">
+      <gazebo reference="${prefix}_diff_unit_link">
+        <selfCollide>false</selfCollide>
+        <material>Gazebo/Orange</material>
+      </gazebo>
+    </xacro:if>
+    <xacro:if value="${warthog_color == 'olive'}">
+      <gazebo reference="${prefix}_diff_unit_link">
+        <selfCollide>false</selfCollide>
+        <!-- TODO we should define a custom gazebo material, but it's not working yet -->
+        <material>Gazebo/Yellow</material>
+      </gazebo>
+    </xacro:if>
+    <xacro:if value="${warthog_color == 'sand'}">
+      <gazebo reference="${prefix}_diff_unit_link">
+        <selfCollide>false</selfCollide>
+        <!-- TODO we should define a custom gazebo material, but it's not working yet -->
+        <material>Gazebo/Yellow</material>
+      </gazebo>
+    </xacro:if>
   </xacro:macro>
   <xacro:diff_unit prefix="left" side="1" left="true"/>

Commit message: Start trying to implement custom colours for the sand & olive materials. No joy so far.

File: warthog_description/urdf/warthog.urdf.xacro (robot description, xacro)
@@ -270,5 +270,8 @@
         <selfCollide>false</selfCollide>
         <!-- TODO we should define a custom gazebo material, but it's not working yet -->
-        <material>Gazebo/Yellow</material>
+        <material>
+          <uri>model://materials/olive.material</uri>
+          <script>Warthog/Olive</script>
+        </material>
       </gazebo>
     </xacro:if>
@@ -277,5 +280,8 @@
         <selfCollide>false</selfCollide>
         <!-- TODO we should define a custom gazebo material, but it's not working yet -->
-        <material>Gazebo/Yellow</material>
+        <material>
+          <uri>model://materials/sand.material</uri>
+          <script>Warthog/Sand</script>
+        </material>
       </gazebo>
     </xacro:if>

Commit message: Remove the material scripts; they weren't working anyway. Add the visual tag around the gazebo material, explicitly define the ambient, diffuse, specular, and emissive properties. Add emissive attributes to the headlights & taillights so they actually show up in the dark

File: warthog_description/urdf/warthog.urdf.xacro (robot description, xacro)
@@ -92,5 +92,5 @@
       <kd value="1.0" />
       <fdir1 value="1 0 0" />
-      <material>Gazebo/Grey</material>
+      <material>Gazebo/DarkGrey</material>
     </gazebo>
     <transmission name="${prefix}_${side}_wheel_trans">
@@ -235,5 +235,12 @@
     </joint>
     <gazebo reference="${prefix}_diff_unit_headlight_link">
-      <material>Gazebo/White</material>
+      <visual>
+        <material>
+          <ambient>0.9 0.9 0.9 1</ambient>
+          <diffuse>0.9 0.9 0.9 1</diffuse>
+          <specular>0.9 0.9 0.9 1</specular>
+          <emissive>0.9 0.9 0.9 1</emissive>
+        </material>
+      </visual>
     </gazebo>
     <link name="${prefix}_diff_unit_taillight_link">
@@ -252,38 +259,24 @@
     </joint>
     <gazebo reference="${prefix}_diff_unit_taillight_link">
-      <material>Gazebo/Red</material>
+      <visual>
+        <material>
+          <ambient>0.9 0 0 1</ambient>
+          <diffuse>0.9 0 0 1</diffuse>
+          <specular>0.9 0 0 1</specular>
+          <emissive>0.9 0 0 1</emissive>
+        </material>
+      </visual>
     </gazebo>
-    <xacro:if value="${warthog_color == 'yellow'}">
-      <gazebo reference="${prefix}_diff_unit_link">
-        <selfCollide>false</selfCollide>
-        <material>Gazebo/Yellow</material>
-      </gazebo>
-    </xacro:if>
-    <xacro:if value="${warthog_color == 'orange'}">
-      <gazebo reference="${prefix}_diff_unit_link">
-        <selfCollide>false</selfCollide>
-        <material>Gazebo/Orange</material>
-      </gazebo>
-    </xacro:if>
-    <xacro:if value="${warthog_color == 'olive'}">
-      <gazebo reference="${prefix}_diff_unit_link">
-        <selfCollide>false</selfCollide>
-        <!-- TODO we should define a custom gazebo material, but it's not working yet -->
+    <gazebo reference="${prefix}_diff_unit_link">
+      <selfCollide>false</selfCollide>
+      <visual>
         <material>
-          <uri>model://materials/olive.material</uri>
-          <script>Warthog/Olive</script>
+          <ambient>${warthog_color_rgba}</ambient>
+          <diffuse>${warthog_color_rgba}</diffuse>
+          <specular>0.1 0.1 0.1 1</specular>
+          <emissive>0 0 0 0</emissive>
         </material>
-      </gazebo>
-    </xacro:if>
-    <xacro:if value="${warthog_color == 'sand'}">
-      <gazebo reference="${prefix}_diff_unit_link">
-        <selfCollide>false</selfCollide>
-        <!-- TODO we should define a custom gazebo material, but it's not working yet -->
-        <material>
-          <uri>model://materials/sand.material</uri>
-          <script>Warthog/Sand</script>
-        </material>
-      </gazebo>
-    </xacro:if>
+      </visual>
+    </gazebo>
   </xacro:macro>
   <xacro:diff_unit prefix="left" side="1" left="true"/>
