Commit message: Added imu link.  Updated inertias for new links

File: warthog_description/urdf/accessories/warthog_arm_mount.urdf.xacro (robot description, xacro)
@@ -16,4 +16,9 @@
         </geometry>
       </collision>
+      <inertial>
+        <origin xyz="0 0 -0.01" rpy="0 0 0"/>
+        <mass value="1.45"/>
+        <xacro:box_inertia m="1.45" x="0.16838" y="0.16838" z="0.02" />
+      </inertial>
     </link>
   </xacro:macro>

File: warthog_description/urdf/accessories/warthog_bulkhead.urdf.xacro (robot description, xacro)
@@ -16,4 +16,9 @@
         </geometry>
       </collision>
+      <inertial>
+        <origin xyz="0.35915 0 -0.6956" rpy="0 0 0"/>
+        <mass value="14.38835"/>
+        <inertia ixx="1.13395" ixy="0.0" ixz="-0.42719" iyy="2.59727" iyz="0.0" izz="3.42344"/>
+      </inertial>
     </link>
     <link name="bulkhead_front_mount_link"/>

File: warthog_description/urdf/warthog.urdf.xacro (robot description, xacro)
@@ -4,5 +4,5 @@
   <material name="dark_grey"><color rgba="0.2 0.2 0.2 1.0" /></material>
   <material name="light_grey"><color rgba="0.4 0.4 0.4 1.0" /></material>
-  <material name="yellow"><color rgba="0.8 0.8 0.0 1.0" /></material>
+  <material name="yellow"><color rgba="0.95 0.816 0.082 1.0" /></material>
   <material name="black"><color rgba="0.15 0.15 0.15 1.0" /></material>
   <material name="white"><color rgba="0.9 0.9 0.9 1.0" /></material>
@@ -84,5 +84,5 @@
           <mesh filename="package://warthog_description/meshes/fenders.stl" />
         </geometry>
-        <material name="yellow"><color rgba="0.8 0.8 0.0 1.0" /></material>
+        <material name="yellow"><color rgba="0.95 0.816 0.082 1.0" /></material>
       </visual>
       <visual>
@@ -124,5 +124,5 @@
   <link name="base_link"></link>
   <joint name="base_link_joint" type="fixed">
-    <origin xyz="0 0 0" rpy="0 0 0" />
+    <origin xyz="0 0 0.025" rpy="0 0 0" />
     <parent link="base_link"/>
     <child link="chassis_link" />
@@ -158,5 +158,5 @@
   <link name="top_chassis_link"></link>
   <joint name="top_link_joint" type="fixed">
-    <origin xyz="0 0 ${chassis_height/2}" rpy="0 0 0" />
+    <origin xyz="0 0 0.27218" rpy="0 0 0" />
     <parent link="chassis_link"/>
     <child link="top_chassis_link" />
@@ -187,7 +187,13 @@
   </link>
   <joint name="diff_link_jnt" type="fixed">
-    <parent link="base_link"/>
+    <parent link="chassis_link"/>
     <child link="diff_link"/>
-    <origin xyz="-0.58245 0 0.27475" rpy="0 0 0" />
+    <origin xyz="-0.5826 0 0.24979" rpy="0 0 0" />
+  </joint>
+  <link name="imu_link" />
+  <joint name="imu_link_joint" type="fixed">
+    <origin xyz="$(optenv WARTHOG_IMU_XYZ 0 0 0)" rpy="$(optenv WARTHOG_IMU_RPY 0 0 0)" />
+    <parent link="chassis_link"/>
+    <child link="imu_link" />
   </joint>
   <!-- Bring in simulation data for Gazebo. -->
